File: elec/pocketPSU_elec_main/user_interface.kicad_sch (KiCad schematic)
At the start: 41 parts, among them J3 Conn_01x12_Pin, SW1 EC11E09244BS, U1 2N7002_C5224215

Commit message: mid-layout
Parts:
- added R21: 10R, Resistor_SMD:R_0402_1005Metric, symbol Device:R_Small
- C1: LCSC Part (none) -> C28323
- C2, C20, C3, C4, C5, C6, C7, C8: LCSC Part (none) -> C15195
- J3, TPCD1, TPCS1, TPENCODER_A1, TPENCODER_B1, TPLEDK1, TPMISO1, TPMOSI1, TPRESET1, TPSCK1: now not fitted
- LED3, LED5: LCSC Part C965864 -> C2290
- R1: value 4.7R -> 10R; LCSC Part (none) -> C25077
- R10, R17, R2, R4, R6, R7, R8, R9: LCSC Part (none) -> C25744
- R19, R20: LCSC Part (none) -> C25076
- R3, R5: value 10K -> 100R; LCSC Part (none) -> C25076
Connections:
- net LEDK: now also R21.1
- net at R1.2, U1.3 (D): now also R21.2

Commit message: finished routing
Parts:
- renumbered BTON-OFF1 to ON-OFF1, BTONCH1 to ON_CH1, BTONCH2 to ON_CH2, U1 to Q1, BTSELCH1 to SEL_CH1, BTSELCH2 to SEL_CH2
Other:
- moved on the sheet: C1
Changed lines of the file:
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@@
 	(wire
 		(pts
-			(xy 186.69 41.91) (xy 186.69 45.72)
+			(xy 208.28 41.91) (xy 208.28 45.72)
 		)
 		(stroke
@@
 	(wire
 		(pts
-			(xy 186.69 33.02) (xy 186.69 36.83)
+			(xy 208.28 33.02) (xy 208.28 36.83)
 		)
 		(stroke
@@
 	(symbol
 		(lib_id "Device:C_Small")
-		(at 186.69 39.37 0)
+		(at 208.28 39.37 0)
 		(unit 1)
 		(exclude_from_sim no)
@@
 		(fields_autoplaced yes)
 		(property "Reference" "C1"
-			(at 189.23 38.1062 0)
+			(at 210.82 38.1062 0)
 			(effects
 				(font
@@
 		)
 		(property "Value" "1uF"
-			(at 189.23 40.6462 0)
+			(at 210.82 40.6462 0)
 			(effects
 				(font
@@
 		)
 		(property "Footprint" "Resistor_SMD:R_0805_2012Metric"
-			(at 186.69 39.37 0)
+			(at 208.28 39.37 0)
 			(effects
 				(font
@@
 		)
 		(property "Datasheet" "~"
-			(at 186.69 39.37 0)
+			(at 208.28 39.37 0)
 			(effects
 				(font
@@
 		)
 		(property "Description" "Unpolarized capacitor, small symbol"
-			(at 186.69 39.37 0)
+			(at 208.28 39.37 0)
 			(effects
 				(font
@@
 		)
 		(property "LCSC Part" "C28323"
-			(at 186.69 39.37 0)
+			(at 208.28 39.37 0)
 			(effects
 				(font
@@
 		(dnp no)
 		(fields_autoplaced yes)
-		(property "Reference" "BTON-OFF1"
+		(property "Reference" "ON-OFF1"
 			(at 181.61 132.08 0)
 			(effects
@@
 			(project "pocketPSU_elec_main"
 				(path "/439011d5-4dd5-4d65-a9bd-b0be402d54a5/cbe29d96-4bd9-4dd2-be02-96003f32f1da"
-					(reference "BTON-OFF1")
+					(reference "ON-OFF1")
 					(unit 1)
 				)
@@
 		(dnp no)
 		(fields_autoplaced yes)
-		(property "Reference" "BTSELCH2"
+		(property "Reference" "SEL_CH2"
 			(at 143.51 132.08 0)
 			(effects
@@
 			(project "pocketPSU_elec_main"
 				(path "/439011d5-4dd5-4d65-a9bd-b0be402d54a5/cbe29d96-4bd9-4dd2-be02-96003f32f1da"
-					(reference "BTSELCH2")
+					(reference "SEL_CH2")
 					(unit 1)
 				)
@@
 		(dnp no)
 		(fields_autoplaced yes)
-		(property "Reference" "BTSELCH1"
+		(property "Reference" "SEL_CH1"
 			(at 67.31 132.08 0)
 			(effects
@@
 			(project "pocketPSU_elec_main"
 				(path "/439011d5-4dd5-4d65-a9bd-b0be402d54a5/cbe29d96-4bd9-4dd2-be02-96003f32f1da"
-					(reference "BTSELCH1")
+					(reference "SEL_CH1")
 					(unit 1)
 				)
@@
 	(symbol
 		(lib_id "power:GND")
-		(at 186.69 45.72 0)
+		(at 208.28 45.72 0)
 		(unit 1)
 		(exclude_from_sim no)
@@
 		(fields_autoplaced yes)
 		(property "Reference" "#PWR06"
-			(at 186.69 52.07 0)
+			(at 208.28 52.07 0)
 			(effects
 				(font
@@
 		)
 		(property "Value" "GND"
-			(at 186.69 50.8 0)
+			(at 208.28 50.8 0)
 			(effects
 				(font
@@
 		)
 		(property "Footprint" ""
-			(at 186.69 45.72 0)
+			(at 208.28 45.72 0)
 			(effects
 				(font
@@
 		)
 		(property "Datasheet" ""
-			(at 186.69 45.72 0)
+			(at 208.28 45.72 0)
 			(effects
 				(font
@@
 		)
 		(property "Description" "Power symbol creates a global label with name \"GND\" , ground"
-			(at 186.69 45.72 0)
+			(at 208.28 45.72 0)
 			(effects
 				(font
@@
 	(symbol
 		(lib_id "power:+3.3V")
-		(at 186.69 33.02 0)
+		(at 208.28 33.02 0)
 		(unit 1)
 		(exclude_from_sim no)
@@
 		(fields_autoplaced yes)
 		(property "Reference" "#PWR07"
-			(at 186.69 36.83 0)
+			(at 208.28 36.83 0)
 			(effects
 				(font
@@
 		)
 		(property "Value" "+3.3V"
-			(at 186.69 27.94 0)
+			(at 208.28 27.94 0)
 			(effects
 				(font
@@
 		)
 		(property "Footprint" ""
-			(at 186.69 33.02 0)
+			(at 208.28 33.02 0)
 			(effects
 				(font
@@
 		)
 		(property "Datasheet" ""
-			(at 186.69 33.02 0)
+			(at 208.28 33.02 0)
 			(effects
 				(font
@@
 		)
 		(property "Description" "Power symbol creates a global label with name \"+3.3V\""
-			(at 186.69 33.02 0)
+			(at 208.28 33.02 0)
 			(effects
 				(font
@@
 		(dnp no)
 		(fields_autoplaced yes)
-		(property "Reference" "BTONCH2"
+		(property "Reference" "ON_CH2"
 			(at 105.41 132.08 0)
 			(effects
@@
 			(project "pocketPSU_elec_main"
 				(path "/439011d5-4dd5-4d65-a9bd-b0be402d54a5/cbe29d96-4bd9-4dd2-be02-96003f32f1da"
-					(reference "BTONCH2")
+					(reference "ON_CH2")
 					(unit 1)
 				)
@@
 		(dnp no)
 		(fields_autoplaced yes)
-		(property "Reference" "BTONCH1"
+		(property "Reference" "ON_CH1"
 			(at 27.94 132.08 0)
 			(effects
@@
 			(project "pocketPSU_elec_main"
 				(path "/439011d5-4dd5-4d65-a9bd-b0be402d54a5/cbe29d96-4bd9-4dd2-be02-96003f32f1da"
-					(reference "BTONCH1")
+					(reference "ON_CH1")
 					(unit 1)
 				)
@@
 		(dnp no)
 		(fields_autoplaced yes)
-		(property "Reference" "U1"
+		(property "Reference" "Q1"
 			(at 153.67 42.5449 0)
 			(effects
@@
 			(project "pocketPSU_elec_main"
 				(path "/439011d5-4dd5-4d65-a9bd-b0be402d54a5/cbe29d96-4bd9-4dd2-be02-96003f32f1da"
-					(reference "U1")
+					(reference "Q1")
 					(unit 1)
 				)
