File: elec/pocketPSU_elec_main/microcontroller.kicad_sch (KiCad schematic)
At the start: 16 parts, among them J1 Header-Male-2.54_1x20, SW3 TS-1187A-B-A-B, SW6 TS-1187A-B-A-B, U2 ESP32-S3-WROOM-1(N16R2), U3 AMS1117-3.3, U5 F.0603.00026/P2-0603B1TS2-06T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

Commit message: mid-layout
Parts:
- added C21, C22: 1uF, Resistor_SMD:R_0805_2012Metric, symbol Device:C_Small
- added C23, C24: 100nF, Capacitor_SMD:C_0805_2012Metric, symbol Device:C_Small
- added R22: 120R, Resistor_SMD:R_0603_1608Metric, symbol Device:R_Small
- added U5: SM04B-GHS-TB(LF)(SN), footprints:CONN-SMD_4P-P1.25_SM04B-GHS-TB-LF-SN, symbol footprints:SM04B-GHS-TB(LF)(SN)
- added U8: TJA1044GT/3Z, footprints:SO-8_L4.9-W3.9-P1.27-LS5.9-BL, symbol footprints:TJA1044GT_3Z
- C10, C9: LCSC Part (none) -> C15850
- C11: LCSC Part (none) -> C49678
- J1: now not fitted
- LED1: renamed from U5; LCSC Part C7496819 -> C2290
- R11, R18: LCSC Part (none) -> C25744
- R15, R16: LCSC Part (none) -> C25076
- renumbered SW3 to SW_BOOT1, SW6 to SW_RESET1
Connections:
- net +3.3V: now also J1.4, J1.5, C23.1, U8.5 (VIO)
- net BLINKY_LED: now also U2.35 (IO42); no longer U2.17 (IO9)
- net BT_ON_CH1: now also U2.9 (IO16); no longer U2.5 (IO5)
- net BT_ON_CH2: now also U2.12 (IO8); no longer U2.7 (IO7)
- net BT_ON_OFF: now also U2.22 (IO14); no longer U2.9 (IO16)
- net BT_SEL_CH1: now also U2.7 (IO7); no longer U2.4 (IO4)
- net BT_SEL_CH2: now also U2.10 (IO17); no longer U2.6 (IO6)
- net CH1_LED: now also U2.8 (IO15); no longer U2.10 (IO17)
- net ENCODER_BT: now also U2.23 (IO21); no longer U2.15 (IO3)
- net GND: now also J1.1, J1.2, J1.20, J1.3, C21.2, C22.2, C23.2, C24.2, U5.4, U5.5, U5.6, U8.2 (GND), U8.8 (STB)
- net IO11: now also J1.17; no longer J1.18, U2.19 (IO11)
- net IO17: now also J1.19; no longer J1.20
- net IO18: now also J1.18; no longer J1.19
- net IO38: now also J1.15; no longer J1.16
- net IO39: now also J1.14; no longer J1.15
- net IO40: now also J1.13; no longer J1.14, U2.33 (IO40)
- net IO41: now also J1.12; no longer J1.13, U2.34 (IO41)
- net IO42: now also J1.11; no longer J1.12, U2.35 (IO42)
- net IO45: now also J1.10; no longer J1.11
- net SCREEN_BACKLIGHT_EN: now also U2.16 (IO46); no longer U2.12 (IO8)
- net SPI_CS: now also U2.18 (IO10); no longer U2.8 (IO15)
- net SPI_DC: now also U2.17 (IO9); no longer U2.18 (IO10)
- net SPI_MISO: now also U2.21 (IO13); no longer U2.20 (IO12)
- net SPI_MOSI: now also U2.19 (IO11); no longer U2.21 (IO13)
- net SPI_RESET: now also U2.15 (IO3); no longer R11.2, SW_RESET1.1 (A), SW_RESET1.2 (B), U2.3 (EN)
- net SPI_SCK: now also U2.20 (IO12); no longer U2.22 (IO14)
- net USB_INT_N: now also U2.6 (IO6); no longer U2.30 (IO37)
- net USB_SCL: now also U2.5 (IO5); no longer U2.29 (IO36)
- net USB_SDA: now also U2.4 (IO4); no longer U2.28 (IO35)
- removed net IO21: J1.17, U2.23 (IO21)
- removed net IO46: J1.10, U2.16 (IO46)
- net VBUS renamed +5V
- net +5V: now also C21.1, C24.1, U5.1, U8.3 (VCC)
- new net: R22.1, U5.2, U8.7 (CANH)
- new net: R22.2, U5.3, U8.6 (CANL)
- new net: C22.1, R11.2, SW_RESET1.1 (A), SW_RESET1.2 (B), U2.3 (EN)
- new net CAN_RX: U2.34 (IO41), U8.4 (RXD)
- new net CAN_TX: U2.33 (IO40), U8.1 (TXD)
Other:
- moved on the sheet: C10, C11, C12, C13, C9, LED1, LED2, R11, R15, R16, SW_RESET1

Commit message: finished routing
Parts:
- added C14, C15: 100nF, Capacitor_SMD:C_0805_2012Metric, symbol Device:C_Small
- added J4: Screw_Terminal_01x02, TerminalBlock_Phoenix:TerminalBlock_Phoenix_MPT-0,5-2-2.54_1x02_P2.54mm_Horizontal, symbol Connector:Screw_Terminal_01x02
- added JP1: SolderJumper_3_Bridged12, Jumper:SolderJumper-3_P1.3mm_Bridged12_RoundedPad1.0x1.5mm_NumberLabels, symbol Jumper:SolderJumper_3_Bridged12
- added U7: TXS0102DCU, Package_SO:VSSOP-8_2.3x2mm_P0.5mm, symbol Logic_LevelTranslator:TXS0102DCU
- renumbered U5 to J5
Connections:
- net IO11 is gone; now on net GND: J1.17
- net IO17 is gone; now on net GND: J1.19
- net IO18 is gone; now on net GND: J1.18
- net IO40 is gone; now on net IO37: J1.13
- net IO41 is gone; now on net IO38: J1.12
- net IO42 is gone; now on net IO39: J1.11
- net +3.3V: now also J1.3, C15.1, JP1.3 (B), U7.3 (VCCA), U7.6 (OE); no longer J1.5
- net +5V: now also J1.5, J1.6, JP1.1 (A)
- net ENCODER_A: now also U2.25 (IO48); no longer U2.39 (IO1)
- net ENCODER_B: now also U2.24 (IO47); no longer U2.38 (IO2)
- net GND: now also C14.2, C15.2, U7.2 (GND); no longer J1.3
- net IO38: no longer J1.15
- net IO39: no longer J1.14
- net IO45: now also J1.16; no longer J1.10
- net RXD0: now also U7.5 (A1); no longer J1.6
- net TXD0: now also U7.4 (A2); no longer J1.7
- net CAN_H: now reaches J5.2, R22.1, U8.7 (CANH)
- net CAN_H: now also J4.2 (Pin_2)
- net CAN_L: now reaches J5.3, R22.2, U8.6 (CANL)
- net CAN_L: now also J4.1 (Pin_1)
- net IO35: now reaches U2.28 (IO35)
- net IO35: now also J1.15
- net IO36: now reaches U2.29 (IO36)
- net IO36: now also J1.14
- net IO37: now reaches U2.30 (IO37)
- net IO47 renamed IO1
- net IO1: now also U2.39 (IO1); no longer U2.24 (IO47)
- net IO48 renamed RX_5V
- net RX_5V: now also U7.8 (B1); no longer U2.25 (IO48)
- new net: C14.1, JP1.2 (C), U7.7 (VCCB)
- new net IO2: J1.10, U2.38 (IO2)
- new net TX_5V: J1.7, U7.1 (B2)
Other:
- moved on the sheet: J5, R22

Commit message: fix erc
Changed lines of the file:
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@@
 	)
 	(junction
+		(at 63.5 149.86)
+		(diameter 0)
+		(color 0 0 0 0)
+	)
+	(junction
 		(at 247.65 73.66)
 		(diameter 0)
@@
 					(unit 1)
 				)
+			)
+		)
+	)
+	(symbol
+		(lib_id "power:PWR_FLAG")
+		(at 63.5 149.86 0)
+		(unit 1)
+		(exclude_from_sim no)
+		(in_bom yes)
+		(on_board yes)
+		(dnp no)
+		(fields_autoplaced yes)
+		(property "Reference" "#FLG01"
+			(at 63.5 147.955 0)
+			(effects
+				(font
+					(size 1.27 1.27)
+				)
+				(hide yes)
+			)
+		)
+		(property "Value" "PWR_FLAG"
+			(at 63.5 144.78 0)
+			(effects
+				(font
+					(size 1.27 1.27)
+				)
+			)
+		)
+		(property "Footprint" ""
+			(at 63.5 149.86 0)
+			(effects
+				(font
+					(size 1.27 1.27)
+				)
+				(hide yes)
+			)
+		)
+		(property "Datasheet" "~"
+			(at 63.5 149.86 0)
+			(effects
+				(font
+					(size 1.27 1.27)
+				)
+				(hide yes)
+			)
+		)
+		(property "Description" "Special symbol for telling ERC where power comes from"
+			(at 63.5 149.86 0)
+			(effects
+				(font
+					(size 1.27 1.27)
+				)
+				(hide yes)
+			)
+		)
+		(pin "1"
+		)
+		(instances
+			(project ""
+				(path "/439011d5-4dd5-4d65-a9bd-b0be402d54a5/725044cc-ecb2-459a-b2bb-596cb099bd1f"
+					(reference "#FLG01")
+					(unit 1)
+				)
