File: elec/pocketPSU_elec_main/usb_input.kicad_sch (KiCad schematic)
At the start: 15 parts, among them J2 Conn_01x03_Pin, U4 FUSB302MPX

Commit message: mid-layout
Parts:
- removed C14: 10uF, Capacitor_SMD:C_0805_2012Metric, symbol Device:C_Small
- removed C15: 100nF, Capacitor_SMD:C_0805_2012Metric, symbol Device:C_Small
- removed J2: Conn_01x03_Pin, Connector_PinHeader_1.27mm:PinHeader_1x03_P1.27mm_Vertical, symbol Connector:Conn_01x03_Pin
- removed LED1: KT-0603R, footprints:LED0603-RD, symbol footprints:KT-0603R
- removed R12: 100R, Resistor_SMD:R_0402_1005Metric, symbol Device:R_Small
- added C25, C26, C27, C28: 47uF, Capacitor_SMD:C_1206_3216Metric, symbol Device:C_Small
- added C29: 10nF, Capacitor_SMD:C_0402_1005Metric, symbol Device:C_Small
- added C30: 4.7uF, Capacitor_SMD:C_1206_3216Metric, symbol Device:C_Small
- added D1: SS14, footprints:SMA_L4.2-W2.6-LS5.3-RD, symbol footprints:SS14
- added L2: NRS6028T220MMGJV, footprints:IND-SMD_L6.0-W6.0, symbol footprints:NRS6028T220MMGJV
- added R23: 10K, Resistor_SMD:R_0402_1005Metric, symbol Device:R_Small
- added R24: 3.3K, Resistor_SMD:R_0402_1005Metric, symbol Device:R_Small
- added U6: TPS5430DDAR, footprints:ESOP-8_L4.9-W3.9-P1.27-LS6.0-TL-EP, symbol footprints:TPS5430DDAR
- C16: LCSC Part (none) -> C28323
- C17: LCSC Part (none) -> C49678
- C18, C19: value 300pF -> 330pF; footprint Capacitor_SMD:C_0805_2012Metric -> Capacitor_SMD:C_0603_1608Metric; LCSC Part (none) -> C1664
- R13, R14: LCSC Part (none) -> C25900
- TPCC1, TPCC2: now not fitted
Connections:
- net USB_VCONN is gone; now on net +3.3V: U4.12 (VCONN), U4.13 (VCONN)
- net +5V: now also C25.1, C26.1, C27.1, C28.1, L2.2, R23.1
- net GND: now also C25.2, C26.2, C27.2, C28.2, C30.2, D1.2 (A), R24.2, U6.6 (GND), U6.9 (PowerPAD)
- net VBUS: now also C30.1, U6.7 (VIN)
- new net: C29.1, D1.1 (K), L2.1, U6.8 (PH)
- new net: R23.2, R24.1, U6.4 (VSENSE)
- new net: C29.2, U6.1 (BOOT)

Commit message: finished routing
Parts:
- added J2: Screw_Terminal_01x02, TerminalBlock_Phoenix:TerminalBlock_Phoenix_MPT-0,5-2-2.54_1x02_P2.54mm_Horizontal, symbol Connector:Screw_Terminal_01x02
Connections:
- net GND: now also J2.2 (Pin_2)
- net VBUS: now also J2.1 (Pin_1)
Changed lines of the file:
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@@
 	)
 	(symbol
+		(lib_id "Connector:Screw_Terminal_01x02")
+		(at 205.74 40.64 0)
+		(mirror x)
+		(unit 1)
+		(exclude_from_sim no)
+		(in_bom yes)
+		(on_board yes)
+		(dnp yes)
+		(property "Reference" "J2"
+			(at 208.28 40.6401 0)
+			(effects
+				(font
+					(size 1.27 1.27)
+				)
+				(justify left)
+			)
+		)
+		(property "Value" "Screw_Terminal_01x02"
+			(at 208.28 38.1001 0)
+			(effects
+				(font
+					(size 1.27 1.27)
+				)
+				(justify left)
+			)
+		)
+		(property "Footprint" "TerminalBlock_Phoenix:TerminalBlock_Phoenix_MPT-0,5-2-2.54_1x02_P2.54mm_Horizontal"
+			(at 205.74 40.64 0)
+			(effects
+				(font
+					(size 1.27 1.27)
+				)
+				(hide yes)
+			)
+		)
+		(property "Datasheet" "~"
+			(at 205.74 40.64 0)
+			(effects
+				(font
+					(size 1.27 1.27)
+				)
+				(hide yes)
+			)
+		)
+		(property "Description" "Generic screw terminal, single row, 01x02, script generated (kicad-library-utils/schlib/autogen/connector/)"
+			(at 205.74 40.64 0)
+			(effects
+				(font
+					(size 1.27 1.27)
+				)
+				(hide yes)
+			)
+		)
+		(pin "1"
+		)
+		(pin "2"
+		)
+		(instances
+			(project "pocketPSU_elec_main"
+				(path "/439011d5-4dd5-4d65-a9bd-b0be402d54a5/6a8f7395-3ccf-431e-bc54-d9f688783b5c"
+					(reference "J2")
+					(unit 1)
+				)
+			)
+		)
+	)
+	(symbol
 		(lib_id "Device:R_Small")
 		(at 46.99 114.3 0)
@@
 	)
 	(symbol
+		(lib_id "power:VBUS")
+		(at 200.66 40.64 90)
+		(unit 1)
+		(exclude_from_sim no)
+		(in_bom yes)
+		(on_board yes)
+		(dnp no)
+		(fields_autoplaced yes)
+		(property "Reference" "#PWR049"
+			(at 204.47 40.64 0)
+			(effects
+				(font
+					(size 1.27 1.27)
+				)
+				(hide yes)
+			)
+		)
+		(property "Value" "VBUS"
+			(at 196.85 40.6399 90)
+			(effects
+				(font
+					(size 1.27 1.27)
+				)
+				(justify left)
+			)
+		)
+		(property "Footprint" ""
+			(at 200.66 40.64 0)
+			(effects
+				(font
+					(size 1.27 1.27)
+				)
+				(hide yes)
+			)
+		)
+		(property "Datasheet" ""
+			(at 200.66 40.64 0)
+			(effects
+				(font
+					(size 1.27 1.27)
+				)
+				(hide yes)
+			)
+		)
+		(property "Description" "Power symbol creates a global label with name \"VBUS\""
+			(at 200.66 40.64 0)
+			(effects
+				(font
+					(size 1.27 1.27)
+				)
+				(hide yes)
+			)
+		)
+		(pin "1"
+		)
+		(instances
+			(project "pocketPSU_elec_main"
+				(path "/439011d5-4dd5-4d65-a9bd-b0be402d54a5/6a8f7395-3ccf-431e-bc54-d9f688783b5c"
+					(reference "#PWR049")
+					(unit 1)
+				)
+			)
+		)
+	)
+	(symbol
 		(lib_id "power:GND")
 		(at 165.1 177.8 0)
@@
 					(unit 1)
 				)
+			)
+		)
+	)
+	(symbol
+		(lib_id "power:GND")
+		(at 200.66 38.1 270)
+		(unit 1)
+		(exclude_from_sim no)
+		(in_bom yes)
+		(on_board yes)
+		(dnp no)
+		(fields_autoplaced yes)
+		(property "Reference" "#PWR055"
+			(at 194.31 38.1 0)
+			(effects
+				(font
+					(size 1.27 1.27)
+				)
+				(hide yes)
+			)
+		)
+		(property "Value" "GND"
+			(at 196.85 38.0999 90)
+			(effects
+				(font
+					(size 1.27 1.27)
+				)
+				(justify right)
+			)
+		)
+		(property "Footprint" ""
+			(at 200.66 38.1 0)
+			(effects
+				(font
+					(size 1.27 1.27)
+				)
+				(hide yes)
+			)
+		)
+		(property "Datasheet" ""
+			(at 200.66 38.1 0)
+			(effects
+				(font
+					(size 1.27 1.27)
+				)
+				(hide yes)
+			)
+		)
+		(property "Description" "Power symbol creates a global label with name \"GND\" , ground"
+			(at 200.66 38.1 0)
+			(effects
+				(font
+					(size 1.27 1.27)
+				)
+				(hide yes)
+			)
+		)
+		(pin "1"
+		)
+		(instances
+			(project "pocketPSU_elec_main"
+				(path "/439011d5-4dd5-4d65-a9bd-b0be402d54a5/6a8f7395-3ccf-431e-bc54-d9f688783b5c"
+					(reference "#PWR055")
+					(unit 1)
+				)

Commit message: fix erc
Connections:
- no-connect marks 0 -> 5
